File: untitled.kicad_sch (KiCad schematic)
At the start: 4 parts, among them K1 SANYOU_SRD_Form_C

Commit message: vdd for bob
Connections:
- net +12V renamed VDD
Changed lines of the file:
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@@
+	(wire
+		(pts
+			(xy 123.19 38.1) (xy 120.65 38.1)
+		)
+		(stroke
+			(width 0)
+			(type default)
+		)
+	)
 	(wire
 		(pts
@@
 	(wire
 		(pts
-			(xy 123.19 39.37) (xy 123.19 43.18)
+			(xy 123.19 38.1) (xy 123.19 43.18)
 		)
 		(stroke
@@
 			)
 			(justify left)
+		)
+	)
+	(hierarchical_label "VDD"
+		(shape input)
+		(at 120.65 38.1 180)
+		(effects
+			(font
+				(size 1.27 1.27)
+			)
+			(justify right)
 		)
 	)
@@
 					(unit 1)
 				)
-			)
-		)
-	)
-	(symbol
-		(lib_id "power:+12V")
-		(at 123.19 39.37 0)
-		(unit 1)
-		(exclude_from_sim no)
-		(in_bom yes)
-		(on_board yes)
-		(dnp no)
-		(property "Reference" "#PWR0101"
-			(at 123.19 43.18 0)
-			(effects
-				(font
-					(size 1.27 1.27)
-				)
-				(hide yes)
-			)
-		)
-		(property "Value" "+12V"
-			(at 123.19 34.29 0)
-			(effects
-				(font
-					(size 1.27 1.27)
-				)
-			)
-		)
-		(property "Footprint" ""
-			(at 123.19 39.37 0)
-			(effects
-				(font
-					(size 1.27 1.27)
-				)
-				(hide yes)
-			)
-		)
-		(property "Datasheet" ""
-			(at 123.19 39.37 0)
-			(effects
-				(font
-					(size 1.27 1.27)
-				)
-				(hide yes)
-			)
-		)
-		(property "Description" "Power symbol creates a global label with name \"+12V\""
-			(at 123.19 39.37 0)
-			(effects
-				(font
-					(size 1.27 1.27)
-				)
-				(hide yes)
-			)
-		)
-		(pin "1"
-		)
-		(instances
-			(project "Ecu"
-				(path "/c4cd18fd-e378-4fd5-a92c-c83bb44c2a2c/028f0b1a-68aa-4c64-b2e2-eb25296278ed"
-					(reference "#PWR020")
-					(unit 1)
-				)
-				(path "/c4cd18fd-e378-4fd5-a92c-c83bb44c2a2c/09c3bd5b-713b-4b99-8447-787d0eeb2502"
-					(reference "#PWR0101")
-					(unit 1)
-				)
-				(path "/c4cd18fd-e378-4fd5-a92c-c83bb44c2a2c/213ba770-bdd5-4bb9-88f8-a2d28d663549"
-					(reference "#PWR019")
-					(unit 1)
-				)
-				(path "/c4cd18fd-e378-4fd5-a92c-c83bb44c2a2c/34b488b3-b8b1-4d7c-a66e-a6064086e74f"
-					(reference "#PWR02")
-					(unit 1)
-				)
-				(path "/c4cd18fd-e378-4fd5-a92c-c83bb44c2a2c/3a4c7325-3aa7-47de-b495-75210654cacb"
-					(reference "#PWR022")
-					(unit 1)
-				)
-				(path "/c4cd18fd-e378-4fd5-a92c-c83bb44c2a2c/3d564a10-b0a1-4dde-a98c-c2ef67c4526a"
-					(reference "#PWR03")
-					(unit 1)
-				)
-				(path "/c4cd18fd-e378-4fd5-a92c-c83bb44c2a2c/5e64c5df-19f9-490c-a3aa-cd876f745353"
-					(reference "#PWR05")
-					(unit 1)
-				)
-				(path "/c4cd18fd-e378-4fd5-a92c-c83bb44c2a2c/7dc4df00-ef54-4c82-8bf0-ac0b1988fde0"
-					(reference "#PWR07")
-					(unit 1)
-				)
-				(path "/c4cd18fd-e378-4fd5-a92c-c83bb44c2a2c/7f24b6c2-2a0e-4638-9f89-536e26bf543d"
-					(reference "#PWR06")
-					(unit 1)
-				)
-				(path "/c4cd18fd-e378-4fd5-a92c-c83bb44c2a2c/82a5b8db-f80a-4d27-b6dc-bec914ad624f"
-					(reference "#PWR08")
-					(unit 1)
-				)
-				(path "/c4cd18fd-e378-4fd5-a92c-c83bb44c2a2c/a7e6400a-9f2f-49d8-8472-a157656f1a40"
-					(reference "#PWR018")
-					(unit 1)
-				)
-				(path "/c4cd18fd-e378-4fd5-a92c-c83bb44c2a2c/b5d223d4-5359-4512-8b76-09bcf12e1558"
-					(reference "#PWR025")
-					(unit 1)
-				)
-				(path "/c4cd18fd-e378-4fd5-a92c-c83bb44c2a2c/be4486e9-e791-4b56-b7a0-e57058418ff1"
-					(reference "#PWR021")
-					(unit 1)
-				)
-				(path "/c4cd18fd-e378-4fd5-a92c-c83bb44c2a2c/cb275ea6-21d8-4fb2-97b2-7dfcc14b8113"
-					(reference "#PWR024")
-					(unit 1)
-				)
-				(path "/c4cd18fd-e378-4fd5-a92c-c83bb44c2a2c/ccb6743f-22ff-4267-8ac5-793811c6edd2"
-					(reference "#PWR04")
-					(unit 1)
-				)
-				(path "/c4cd18fd-e378-4fd5-a92c-c83bb44c2a2c/df760b5e-b648-4a6a-9551-94014ac70c31"
-					(reference "#PWR023")
-					(unit 1)
-				)
