File: Ecu.kicad_pcb (KiCad board)
At the start: 2 copper layers, 350 x 210 mm, 77 parts, among them J1 Barrel_Jack_MountingPin, J2 DE9_Pins, J3 DE9_Pins, J4 DE9_Pins, J5 DE9_Pins, J6 DE9_Pins, K1 SANYOU_SRD_Form_C, K10 SANYOU_SRD_Form_C, K11 SANYOU_SRD_Form_C, K12 SANYOU_SRD_Form_C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

Commit message: adding pcb
Parts:
- added J7: Conn_01x03_Pin, Connector_PinHeader_1.00mm:PinHeader_1x03_P1.00mm_Vertical, F.Cu at (766.5, 136.0)
Connections:
- D18 pad 1: +12V -> /CINY10/VDD
- D20 pad 1: +12V -> /CINY10/VDD
- D22 pad 1: +12V -> /CINY10/VDD
- D24 pad 1: +12V -> /CINY10/VDD
- D26 pad 1: +12V -> /CINY12/VDD
- D28 pad 1: +12V -> /CINY13/VDD
- D30 pad 1: +12V -> /CINY14/VDD
- D32 pad 1: +12V -> /CINY10/VDD
- K10 pad 1: +12V -> /CINY10/VDD
- K10 pad 2: +12V -> /CINY10/VDD
- K11 pad 1: +12V -> /CINY10/VDD
- K11 pad 2: +12V -> /CINY10/VDD
- K12 pad 1: +12V -> /CINY10/VDD
- K12 pad 2: +12V -> /CINY10/VDD
- K13 pad 1: +12V -> /CINY12/VDD
- K13 pad 2: +12V -> /CINY12/VDD
- K14 pad 1: +12V -> /CINY13/VDD
- K14 pad 2: +12V -> /CINY13/VDD
- K15 pad 1: +12V -> /CINY14/VDD
- K15 pad 2: +12V -> /CINY14/VDD
- K16 pad 1: +12V -> /CINY10/VDD
- K16 pad 2: +12V -> /CINY10/VDD
- K9 pad 1: +12V -> /CINY10/VDD
- K9 pad 2: +12V -> /CINY10/VDD
- R10 pad 1: +12V -> /CINY10/VDD
- R11 pad 1: +12V -> /CINY10/VDD
- R12 pad 1: +12V -> /CINY10/VDD
- R13 pad 1: +12V -> /CINY12/VDD
- R14 pad 1: +12V -> /CINY13/VDD
- R15 pad 1: +12V -> /CINY14/VDD
- R16 pad 1: +12V -> /CINY10/VDD
- R9 pad 1: +12V -> /CINY10/VDD
Routing:
- net +12V: track 0.00 -> 501.6 mm
- net /CINY10/VDD: track 0.00 -> 242.0 mm
- net VREF: track 0.00 -> 114.9 mm
- net /BOUT3: track 0.00 -> 72.6 mm, vias 0 -> 1
- net /OY1: track 0.00 -> 66.2 mm, vias 0 -> 1
- net /BOUT6: track 0.00 -> 63.6 mm
- net /BOUT4: track 0.00 -> 61.5 mm, vias 0 -> 1
- net /STPS: track 0.00 -> 61.0 mm
- net /OY7: track 0.00 -> 59.4 mm, vias 0 -> 1
- net /OY4: track 0.00 -> 53.5 mm
- net /OY2: track 0.00 -> 52.3 mm
- net /OY5: track 0.00 -> 51.6 mm, vias 0 -> 1
- net /BOUT8: track 0.00 -> 51.2 mm
- net /BOUT1: track 0.00 -> 51.2 mm, vias 0 -> 1
- net /SMAP: track 0.00 -> 49.0 mm, vias 0 -> 1
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- added copper zone on B.Cu, net GND
- added copper zone on F.Cu, net GND
Other:
- board text added: "+12V"
- board text added: "BOBINAS"
- board text added: "GND"
- board text added: "INYECTORES"

Commit message: trace curve
Parts:
- added BNCX1: Conn_01x02_Pin, Connector_PinHeader_1.00mm:PinHeader_1x02_P1.00mm_Vertical, F.Cu at (788.1, 230.6)
- added BNCY1: Conn_01x02_Pin, Connector_PinHeader_1.00mm:PinHeader_1x02_P1.00mm_Vertical, F.Cu at (791.4, 230.6)
- added C1: C, Capacitor_SMD:C_1206_3216Metric, F.Cu at (819.3, 221.4)
- added C2: C, Capacitor_SMD:C_1206_3216Metric, F.Cu at (819.3, 224.8)
- added C3: C, Capacitor_SMD:C_1206_3216Metric, F.Cu at (819.3, 228.1)
- added C4: C, Capacitor_SMD:C_1206_3216Metric, F.Cu at (819.3, 231.5)
- added DUT1: Conn_01x02_Pin, Connector_PinHeader_1.00mm:PinHeader_1x02_P1.00mm_Vertical, F.Cu at (794.8, 230.6)
- added Q1: 2N3904, Package_TO_SOT_THT:TO-92_Inline, F.Cu at (818.4, 236.4)
- added R17: R, Resistor_SMD:R_1206_3216Metric, F.Cu at (808.0, 221.4)
- added R18: R, Resistor_SMD:R_1206_3216Metric, F.Cu at (808.0, 224.7)
- added R19: R, Resistor_SMD:R_1206_3216Metric, F.Cu at (808.0, 228.0)
- added R20: R, Resistor_SMD:R_1206_3216Metric, F.Cu at (808.0, 231.3)
- added R21: R, Resistor_SMD:R_1206_3216Metric, F.Cu at (808.0, 234.7)
- added R22: R, Resistor_SMD:R_1206_3216Metric, F.Cu at (808.0, 238.0)
- added R23: R, Resistor_SMD:R_1206_3216Metric, F.Cu at (813.6, 221.4)
- added R24: R, Resistor_SMD:R_1206_3216Metric, F.Cu at (813.6, 224.7)
- added R25: R, Resistor_SMD:R_1206_3216Metric, F.Cu at (813.6, 228.0)
- added R26: R, Resistor_SMD:R_1206_3216Metric, F.Cu at (813.6, 231.3)
- added R27: R, Resistor_SMD:R_1206_3216Metric, F.Cu at (813.6, 234.7)
- added U2: MCP6002-xMC, Package_DFN_QFN:DFN-8-1EP_3x2mm_P0.5mm_EP1.75x1.45mm, F.Cu at (825.0, 221.7)
- moved D19 86.5 mm to (739.3, 230.3)
- moved D20 86.5 mm to (732.4, 230.9)
- moved R10 86.5 mm to (744.9, 230.3)
- moved D17 74.1 mm to (800.7, 161.5)
- moved R9 74.1 mm to (806.3, 161.5)
- moved D18 74.1 mm to (793.8, 162.1)
- moved K9 73.7 mm to (791.8, 151.3)
- moved J6 67.7 mm to (739.2, 166.8), turned to 0 degrees
- moved K10 65.0 mm to (730.4, 220.2)
- moved D29 63.6 mm to (777.5, 208.5)
- moved D30 63.6 mm to (770.6, 209.1)
- moved R15 63.6 mm to (783.1, 208.5)
- moved D24 62.1 mm to (793.8, 185.6)
- moved D23 62.1 mm to (800.7, 185.0)
- moved R12 62.1 mm to (806.3, 185.0)
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Connections:
- D18 pad 1: /CINY10/VDD -> /CINY8/VDD
- D20 pad 1: /CINY10/VDD -> /VD
- D24 pad 1: /CINY10/VDD -> /VD
- D26 pad 1: /CINY12/VDD -> /VD
- D28 pad 1: /CINY13/VDD -> /VD
- D30 pad 1: /CINY14/VDD -> /VD
- D32 pad 1: /CINY10/VDD -> /VD
- J2 pad 1: /IY1 -> unconnected-(J2-Pad1)
- J2 pad 2: /<NO NET> -> unconnected-(J2-Pad2)
- J2 pad 3: /IY3 -> unconnected-(J2-Pad3)
- J2 pad 4: /IY4 -> unconnected-(J2-Pad4)
- J2 pad 6: /OY1 -> unconnected-(J2-Pad6)
- J2 pad 7: /OY2 -> unconnected-(J2-Pad7)
- J2 pad 8: /OY3 -> unconnected-(J2-Pad8)
- J2 pad 9: /OY4 -> unconnected-(J2-Pad9)
- J3 pad 1: /IY5 -> /IY1
- J3 pad 2: /IY6 -> /IY3
- J3 pad 3: /IY7 -> /IY5
- J3 pad 4: /IY8 -> /IY7
- J3 pad 6: /OY5 -> /<NO NET>
- J3 pad 7: /OY6 -> /IY4
- J3 pad 8: /OY7 -> /IY6
- J3 pad 9: /OY8 -> /IY8
- J4 pad 3: unconnected-(J4-Pad3) -> /STPS
- J4 pad 8: /STPS -> /SMAF
- J4 pad 9: /SMAF -> unconnected-(J4-Pad9)
- J5 pad 2: /<NO NET> -> /BOB3
- J5 pad 3: /BOB3 -> /BOB5
- J5 pad 4: /BOB4 -> /BOB7
- J5 pad 6: /BOUT1 -> /<NO NET>
- J5 pad 7: /BOUT2 -> /BOB4
- J5 pad 8: /BOUT3 -> /BOB6
- J5 pad 9: /BOUT4 -> /BOB8
- J6 pad 1: /BOB5 -> unconnected-(J6-Pad1)
- J6 pad 2: /BOB6 -> unconnected-(J6-Pad2)
- J6 pad 3: /BOB7 -> unconnected-(J6-Pad3)
- J6 pad 4: /BOB8 -> unconnected-(J6-Pad4)
- J6 pad 6: /BOUT5 -> unconnected-(J6-Pad6)
- J6 pad 7: /BOUT6 -> unconnected-(J6-Pad7)
- J6 pad 8: /BOUT7 -> unconnected-(J6-Pad8)
- J6 pad 9: /BOUT8 -> unconnected-(J6-Pad9)
- J7 pad 2: /CINY10/VDD -> /VD
- K10 pad 1: /CINY10/VDD -> /VD
- K10 pad 2: /CINY10/VDD -> /VD
- K12 pad 1: /CINY10/VDD -> /VD
- K12 pad 2: /CINY10/VDD -> /VD
- K13 pad 1: /CINY12/VDD -> /VD
- K13 pad 2: /CINY12/VDD -> /VD
- K14 pad 1: /CINY13/VDD -> /VD
- K14 pad 2: /CINY13/VDD -> /VD
- K15 pad 1: /CINY14/VDD -> /VD
- K15 pad 2: /CINY14/VDD -> /VD
- K16 pad 1: /CINY10/VDD -> /VD
- K16 pad 2: /CINY10/VDD -> /VD
- K9 pad 1: /CINY10/VDD -> /CINY8/VDD
- K9 pad 2: /CINY10/VDD -> /CINY8/VDD
- R10 pad 1: /CINY10/VDD -> /VD
- R12 pad 1: /CINY10/VDD -> /VD
- R13 pad 1: /CINY12/VDD -> /VD
- R14 pad 1: /CINY13/VDD -> /VD
- R15 pad 1: /CINY14/VDD -> /VD
- R16 pad 1: /CINY10/VDD -> /VD
- R9 pad 1: /CINY10/VDD -> /CINY8/VDD
Routing:
- net /CINY10/VDD: track 242.0 -> 0.00 mm
- net +12V: track 501.6 -> 397.9 mm
- net /BOUT3: track 72.6 -> 0.00 mm, vias 1 -> 0
- net /OY1: track 66.2 -> 0.00 mm, vias 1 -> 0
- net /BOUT6: track 63.6 -> 0.00 mm
- net /BOUT4: track 61.5 -> 0.00 mm, vias 1 -> 0
- net /OY7: track 59.4 -> 0.00 mm, vias 1 -> 0
- net /OY4: track 53.5 -> 0.00 mm
- net /OY2: track 52.3 -> 0.00 mm
- net /OY5: track 51.6 -> 0.00 mm, vias 1 -> 0
- net /BOUT8: track 51.2 -> 0.00 mm
- net /BOUT1: track 51.2 -> 0.00 mm, vias 1 -> 0
- net /BOUT5: track 42.8 -> 0.00 mm
- net /OY6: track 42.1 -> 0.00 mm, vias 1 -> 0
- net /BOUT7: track 38.5 -> 0.00 mm
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Other:
- board text added: "ECT"
- board text added: "IAT"
- board text added: "MAF"
- board text added: "MAP"
- board text added: "O2"
- board text added: "TPS"
- board text removed: "+12V"
- board text removed: "BOBINAS"
- board text removed: "GND"
