File: Ecu.kicad_sch (KiCad schematic)
At the start: 7 parts, among them J1 Barrel_Jack_MountingPin, J2 DE9_Pins, J3 DE9_Pins, J4 DE9_Pins, J5 DE9_Pins, J6 DE9_Pins, U1 L7805

Commit message: vdd for bob
Other:
- sheet CINY ports: added VDD; removed none
- sheet CINY1 ports: added VDD; removed none
- sheet CINY10 ports: added VDD; removed none
- sheet CINY11 ports: added VDD; removed none
- sheet CINY12 ports: added VDD; removed none
- sheet CINY13 ports: added VDD; removed none
- sheet CINY14 ports: added VDD; removed none
- sheet CINY15 ports: added VDD; removed none
- sheet CINY2 ports: added VDD; removed none
- sheet CINY3 ports: added VDD; removed none
- sheet CINY4 ports: added VDD; removed none
- sheet CINY5 ports: added VDD; removed none
- sheet CINY6 ports: added VDD; removed none
- sheet CINY7 ports: added VDD; removed none
- sheet CINY8 ports: added VDD; removed none
- sheet CINY9 ports: added VDD; removed none

Commit message: adding pcb
Parts:
- added J7: Conn_01x03_Pin, Connector_PinHeader_1.00mm:PinHeader_1x03_P1.00mm_Vertical, symbol Connector:Conn_01x03_Pin
Connections:
- net +12V: now also J7.3 (Pin_3)
- net CINY10/VDD: now also J7.2 (Pin_2)
- net GND: now also J7.1 (Pin_1)

Commit message: trace curve
Connections:
- net BOB3: now also J5.2; no longer J5.3
- net BOB4: now also J5.7; no longer J5.4
- net BOB5: now also J5.3; no longer J6.1
- net BOB6: now also J5.8; no longer J6.2
- net BOB7: now also J5.4; no longer J6.3
- net BOB8: now also J5.9; no longer J6.4
- net BOUT1: no longer J5.6
- net BOUT2: no longer J5.7
- net BOUT3: no longer J5.8
- net BOUT4: no longer J5.9
- net BOUT5: no longer J6.6
- net BOUT6: no longer J6.7
- net BOUT7: no longer J6.8
- net BOUT8: no longer J6.9
- net CINY10/VDD: no longer J7.2 (Pin_2)
- net IY1: now also J3.1; no longer J2.1
- net IY3: now also J3.2; no longer J2.3
- net IY4: now also J3.7; no longer J2.4
- net IY5: now also J3.3; no longer J3.1
- net IY6: now also J3.8; no longer J3.2
- net IY7: now also J3.4; no longer J3.3
- net IY8: now also J3.9; no longer J3.4
- net OY1: no longer J2.6
- net OY2: no longer J2.7
- net OY3: no longer J2.8
- net OY4: no longer J2.9
- net OY5: no longer J3.6
- net OY6: no longer J3.7
- net OY7: no longer J3.8
- net OY8: no longer J3.9
- net SMAF: now also J4.8; no longer J4.9
- net STPS: now also J4.3; no longer J4.8
- net at J2.2: no longer names the net of J2.2
- net at J2.2: no longer J5.2
- new net: J3.6, J5.6
- new net VD: J7.2 (Pin_2)
Other:
- added sheet Trace Curve (trace_curve.kicad_sch)
- moved on the sheet: J1, J2, J3, J4, J5, J6, J7, U1

Commit message: new structure
Parts:
- removed J2, J3, J4, J5, J6: DE9_Pins, Connector_Dsub:DSUB-9_Pins_Horizontal_P2.77x2.54mm_EdgePinOffset9.40mm, symbol Connector:DE9_Pins
- removed J7: Conn_01x03_Pin, Connector_PinHeader_1.00mm:PinHeader_1x03_P1.00mm_Vertical, symbol Connector:Conn_01x03_Pin
Other:
- removed sheet CINY
- removed sheet CINY1
- removed sheet CINY10
- removed sheet CINY11
- removed sheet CINY12
- removed sheet CINY13
- removed sheet CINY14
- removed sheet CINY15
- removed sheet CINY2
- removed sheet CINY3
- removed sheet CINY4
- removed sheet CINY5
- removed sheet CINY6
- removed sheet CINY7
- removed sheet CINY8
- removed sheet CINY9
- removed sheet SIM
- removed sheet SIM1
- removed sheet SIM2
- removed sheet SIM3
- removed sheet SIM4
- removed sheet SIM5
- added sheet Diode bridge (diode_bridge.kicad_sch)
- added sheet Led Indicator (led_indicator.kicad_sch)
- added sheet Relay indicator (relay_indicator.kicad_sch)
- added sheet Voltage simulator (voltage_simulator.kicad_sch)
- moved on the sheet: J1, U1
