File: relay_indicator.kicad_sch (KiCad schematic)
At the start: 4 parts, among them K1 SANYOU_SRD_Form_C

Commit message: new structure
Parts:
- removed D2: D_Schottky, Diode_SMD:D_SMA, symbol Device:D_Schottky
- added D?: D_TVS, symbol Device:D_TVS
- added D?: LED, LED_SMD:LED_1206_3216Metric, symbol Device:LED
- renumbered D1 to D?, K1 to K?, R1 to R?
Connections:
- net INPUT: now reaches D?.1 (K), K?.5
- net INPUT: now also D?.1 (A1), D?.2 (A)
- net at D?.2 (A), R?.2: now also D?.1 (K)
- net OUTY renamed DRV_OUT
- net VDD renamed COIL_RAIL
- net COIL_RAIL: now also D?.2 (A2)
Other:
- moved on the sheet: D?, K?, R?
