File: trace_curve.kicad_sch (KiCad schematic)
At the start: 20 parts, among them Q1 2N3904, U2 MCP6002-xMC

Commit message: new structure
Parts:
- removed unit 3 of U2
- added U1: MCP6002-xMC, Package_DFN_QFN:DFN-8-1EP_3x2mm_P0.5mm_EP1.75x1.45mm, symbol Amplifier_Operational:MCP6002-xMC
Changed lines of the file:
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@@
 		)
 		(instances
+			(project "trace_curve"
+				(path "/7b27ef15-3887-4fdd-ab7f-e6e60a80fdbd"
+					(reference "#PWR?")
+					(unit 1)
+				)
+			)
 			(project "Ecu"
 				(path "/c4cd18fd-e378-4fd5-a92c-c83bb44c2a2c/947ca78a-d82d-42f0-b91e-0681d89f1af6"
@@
 		)
 		(instances
+			(project "trace_curve"
+				(path "/7b27ef15-3887-4fdd-ab7f-e6e60a80fdbd"
+					(reference "R?")
+					(unit 1)
+				)
+			)
 			(project ""
 				(path "/c4cd18fd-e378-4fd5-a92c-c83bb44c2a2c/947ca78a-d82d-42f0-b91e-0681d89f1af6"
@@
 		(lib_id "Amplifier_Operational:MCP6002-xMC")
 		(at 256.54 39.37 0)
-		(unit 3)
-		(exclude_from_sim no)
-		(in_bom yes)
-		(on_board yes)
-		(dnp no)
-		(fields_autoplaced yes)
-		(property "Reference" "U2"
+		(unit 1)
+		(exclude_from_sim no)
+		(in_bom yes)
+		(on_board yes)
+		(dnp no)
+		(fields_autoplaced yes)
+		(property "Reference" "U?"
 			(at 255.27 38.0999 0)
 			(effects
@@
 			)
 		)
-		(pin "2"
+		(pin "8"
+		)
+		(pin "6"
+		)
+		(pin "5"
 		)
 		(pin "3"
 		)
-		(pin "5"
-		)
-		(pin "6"
+		(pin "1"
+		)
+		(pin "9"
+		)
+		(pin "7"
+		)
+		(pin "2"
 		)
 		(pin "4"
 		)
-		(pin "8"
-		)
-		(pin "7"
-		)
-		(pin "1"
-		)
-		(pin "9"
-		)
-		(instances
-			(project ""
-				(path "/c4cd18fd-e378-4fd5-a92c-c83bb44c2a2c/947ca78a-d82d-42f0-b91e-0681d89f1af6"
-					(reference "U2")
+		(instances
+			(project ""
+				(path "/7b27ef15-3887-4fdd-ab7f-e6e60a80fdbd"
+					(reference "U1")
 					(unit 3)
+				)
+			)
+			(project "Ecu"
+				(path "/c4cd18fd-e378-4fd5-a92c-c83bb44c2a2c/947ca78a-d82d-42f0-b91e-0681d89f1af6"
+					(reference "U?")
+					(unit 1)
 				)
 			)
@@
 		)
 		(instances
+			(project "trace_curve"
+				(path "/7b27ef15-3887-4fdd-ab7f-e6e60a80fdbd"
+					(reference "R?")
+					(unit 1)
+				)
+			)
 			(project ""
 				(path "/c4cd18fd-e378-4fd5-a92c-c83bb44c2a2c/947ca78a-d82d-42f0-b91e-0681d89f1af6"
@@
 		)
 		(instances
+			(project "trace_curve"
+				(path "/7b27ef15-3887-4fdd-ab7f-e6e60a80fdbd"
+					(reference "R?")
+					(unit 1)
+				)
+			)
 			(project ""
 				(path "/c4cd18fd-e378-4fd5-a92c-c83bb44c2a2c/947ca78a-d82d-42f0-b91e-0681d89f1af6"
@@
 		)
 		(instances
+			(project "trace_curve"
+				(path "/7b27ef15-3887-4fdd-ab7f-e6e60a80fdbd"
+					(reference "U?")
+					(unit 1)
+				)
+			)
 			(project ""
 				(path "/c4cd18fd-e378-4fd5-a92c-c83bb44c2a2c/947ca78a-d82d-42f0-b91e-0681d89f1af6"
@@
 		)
 		(instances
+			(project "trace_curve"
+				(path "/7b27ef15-3887-4fdd-ab7f-e6e60a80fdbd"
+					(reference "U?")
+					(unit 1)
+				)
+			)
 			(project ""
 				(path "/c4cd18fd-e378-4fd5-a92c-c83bb44c2a2c/947ca78a-d82d-42f0-b91e-0681d89f1af6"
@@
 		)
 		(instances
+			(project "trace_curve"
+				(path "/7b27ef15-3887-4fdd-ab7f-e6e60a80fdbd"
+					(reference "C?")
+					(unit 1)
+				)
+			)
 			(project ""
 				(path "/c4cd18fd-e378-4fd5-a92c-c83bb44c2a2c/947ca78a-d82d-42f0-b91e-0681d89f1af6"
@@
 		)
 		(instances
+			(project "trace_curve"
+				(path "/7b27ef15-3887-4fdd-ab7f-e6e60a80fdbd"
+					(reference "R?")
+					(unit 1)
+				)
+			)
 			(project ""
 				(path "/c4cd18fd-e378-4fd5-a92c-c83bb44c2a2c/947ca78a-d82d-42f0-b91e-0681d89f1af6"
@@
 		)
 		(instances
+			(project "trace_curve"
+				(path "/7b27ef15-3887-4fdd-ab7f-e6e60a80fdbd"
+					(reference "C?")
+					(unit 1)
+				)
+			)
 			(project ""
 				(path "/c4cd18fd-e378-4fd5-a92c-c83bb44c2a2c/947ca78a-d82d-42f0-b91e-0681d89f1af6"
@@
 		)
 		(instances
+			(project "trace_curve"
+				(path "/7b27ef15-3887-4fdd-ab7f-e6e60a80fdbd"
+					(reference "#PWR?")
+					(unit 1)
+				)
+			)
 			(project "Ecu"
 				(path "/c4cd18fd-e378-4fd5-a92c-c83bb44c2a2c/947ca78a-d82d-42f0-b91e-0681d89f1af6"
@@
 		)
 		(instances
+			(project "trace_curve"
+				(path "/7b27ef15-3887-4fdd-ab7f-e6e60a80fdbd"
+					(reference "R?")
+					(unit 1)
+				)
+			)
 			(project ""
 				(path "/c4cd18fd-e378-4fd5-a92c-c83bb44c2a2c/947ca78a-d82d-42f0-b91e-0681d89f1af6"
@@
 		)
 		(instances
+			(project "trace_curve"
+				(path "/7b27ef15-3887-4fdd-ab7f-e6e60a80fdbd"
+					(reference "C?")
+					(unit 1)
+				)
+			)
 			(project ""
 				(path "/c4cd18fd-e378-4fd5-a92c-c83bb44c2a2c/947ca78a-d82d-42f0-b91e-0681d89f1af6"
@@
 		)
 		(instances
+			(project "trace_curve"
+				(path "/7b27ef15-3887-4fdd-ab7f-e6e60a80fdbd"
+					(reference "R?")
+					(unit 1)
+				)
+			)
 			(project ""
 				(path "/c4cd18fd-e378-4fd5-a92c-c83bb44c2a2c/947ca78a-d82d-42f0-b91e-0681d89f1af6"
@@
 		)
 		(instances
+			(project "trace_curve"
+				(path "/7b27ef15-3887-4fdd-ab7f-e6e60a80fdbd"
+					(reference "#PWR?")
+					(unit 1)
+				)
+			)
 			(project "Ecu"
 				(path "/c4cd18fd-e378-4fd5-a92c-c83bb44c2a2c/947ca78a-d82d-42f0-b91e-0681d89f1af6"
@@
 		)
 		(instances
+			(project "trace_curve"
+				(path "/7b27ef15-3887-4fdd-ab7f-e6e60a80fdbd"
+					(reference "#PWR?")
+					(unit 1)
+				)
+			)
 			(project "Ecu"
 				(path "/c4cd18fd-e378-4fd5-a92c-c83bb44c2a2c/947ca78a-d82d-42f0-b91e-0681d89f1af6"
@@
 		)
 		(instances
+			(project "trace_curve"
+				(path "/7b27ef15-3887-4fdd-ab7f-e6e60a80fdbd"
+					(reference "#PWR?")
+					(unit 1)
+				)
+			)
 			(project "Ecu"
 				(path "/c4cd18fd-e378-4fd5-a92c-c83bb44c2a2c/947ca78a-d82d-42f0-b91e-0681d89f1af6"
@@
 		)
 		(instances
+			(project "trace_curve"
+				(path "/7b27ef15-3887-4fdd-ab7f-e6e60a80fdbd"
+					(reference "R?")
+					(unit 1)
+				)
+			)
 			(project ""
 				(path "/c4cd18fd-e378-4fd5-a92c-c83bb44c2a2c/947ca78a-d82d-42f0-b91e-0681d89f1af6"
@@
 		)
 		(instances
+			(project "trace_curve"
+				(path "/7b27ef15-3887-4fdd-ab7f-e6e60a80fdbd"
+					(reference "#PWR?")
+					(unit 1)
+				)
+			)
 			(project ""
 				(path "/c4cd18fd-e378-4fd5-a92c-c83bb44c2a2c/947ca78a-d82d-42f0-b91e-0681d89f1af6"
@@
 		)
 		(instances
+			(project "trace_curve"
+				(path "/7b27ef15-3887-4fdd-ab7f-e6e60a80fdbd"
+					(reference "DUT?")
+					(unit 1)
+				)
+			)
 			(project ""
 				(path "/c4cd18fd-e378-4fd5-a92c-c83bb44c2a2c/947ca78a-d82d-42f0-b91e-0681d89f1af6"
@@
 		)
 		(instances
+			(project "trace_curve"
+				(path "/7b27ef15-3887-4fdd-ab7f-e6e60a80fdbd"
+					(reference "BNCX?")
+					(unit 1)
+				)
+			)
 			(project ""
 				(path "/c4cd18fd-e378-4fd5-a92c-c83bb44c2a2c/947ca78a-d82d-42f0-b91e-0681d89f1af6"
@@
 		)
 		(instances
+			(project "trace_curve"
+				(path "/7b27ef15-3887-4fdd-ab7f-e6e60a80fdbd"
+					(reference "R?")
+					(unit 1)
+				)
+			)
 			(project ""
 				(path "/c4cd18fd-e378-4fd5-a92c-c83bb44c2a2c/947ca78a-d82d-42f0-b91e-0681d89f1af6"
@@
 		)
 		(instances
+			(project "trace_curve"
+				(path "/7b27ef15-3887-4fdd-ab7f-e6e60a80fdbd"
+					(reference "Q?")
+					(unit 1)
+				)
+			)
 			(project ""
 				(path "/c4cd18fd-e378-4fd5-a92c-c83bb44c2a2c/947ca78a-d82d-42f0-b91e-0681d89f1af6"
@@
 		)
 		(instances
+			(project "trace_curve"
+				(path "/7b27ef15-3887-4fdd-ab7f-e6e60a80fdbd"
+					(reference "BNCY?")
+					(unit 1)
+				)
+			)
 			(project ""
 				(path "/c4cd18fd-e378-4fd5-a92c-c83bb44c2a2c/947ca78a-d82d-42f0-b91e-0681d89f1af6"
@@
 		)
 		(instances
+			(project "trace_curve"
+				(path "/7b27ef15-3887-4fdd-ab7f-e6e60a80fdbd"
+					(reference "R?")
+					(unit 1)
+				)
+			)
 			(project ""
 				(path "/c4cd18fd-e378-4fd5-a92c-c83bb44c2a2c/947ca78a-d82d-42f0-b91e-0681d89f1af6"
@@
 		)
 		(instances
+			(project "trace_curve"
+				(path "/7b27ef15-3887-4fdd-ab7f-e6e60a80fdbd"
+					(reference "R?")
+					(unit 1)
+				)
+			)
 			(project ""
 				(path "/c4cd18fd-e378-4fd5-a92c-c83bb44c2a2c/947ca78a-d82d-42f0-b91e-0681d89f1af6"
@@
 		)
 		(instances
+			(project "trace_curve"
+				(path "/7b27ef15-3887-4fdd-ab7f-e6e60a80fdbd"
+					(reference "R?")
+					(unit 1)
+				)
+			)
 			(project ""
 				(path "/c4cd18fd-e378-4fd5-a92c-c83bb44c2a2c/947ca78a-d82d-42f0-b91e-0681d89f1af6"
@@
 		)
 		(instances
+			(project "trace_curve"
+				(path "/7b27ef15-3887-4fdd-ab7f-e6e60a80fdbd"
+					(reference "C?")
+					(unit 1)
+				)
+			)
 			(project ""
 				(path "/c4cd18fd-e378-4fd5-a92c-c83bb44c2a2c/947ca78a-d82d-42f0-b91e-0681d89f1af6"
@@
 		)
 	)
+	(sheet_instances
+		(path "/"
+			(page "1")
+		)
+	)
+	(embedded_fonts no)
 )
