File: voltage_simulator.kicad_sch (KiCad schematic)
At the start: 1 part

Commit message: new structure
Other:
- moved on the sheet: RV1
Changed lines of the file:
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@@
 	(wire
 		(pts
-			(xy 53.34 46.99) (xy 53.34 53.34)
-		)
-		(stroke
-			(width 0)
-			(type default)
-		)
-	)
-	(wire
-		(pts
-			(xy 46.99 34.29) (xy 53.34 34.29)
-		)
-		(stroke
-			(width 0)
-			(type default)
-		)
-	)
-	(wire
-		(pts
-			(xy 57.15 43.18) (xy 64.77 43.18)
-		)
-		(stroke
-			(width 0)
-			(type default)
-		)
-	)
-	(wire
-		(pts
-			(xy 53.34 34.29) (xy 53.34 39.37)
+			(xy 88.9 62.23) (xy 88.9 68.58)
+		)
+		(stroke
+			(width 0)
+			(type default)
+		)
+	)
+	(wire
+		(pts
+			(xy 82.55 49.53) (xy 88.9 49.53)
+		)
+		(stroke
+			(width 0)
+			(type default)
+		)
+	)
+	(wire
+		(pts
+			(xy 88.9 49.53) (xy 88.9 54.61)
+		)
+		(stroke
+			(width 0)
+			(type default)
+		)
+	)
+	(wire
+		(pts
+			(xy 92.71 58.42) (xy 100.33 58.42)
 		)
 		(stroke
@@
 	(global_label "VREF"
 		(shape input)
-		(at 46.99 34.29 180)
+		(at 82.55 49.53 180)
 		(fields_autoplaced yes)
 		(effects
@@
 		)
 		(property "Intersheetrefs" "${INTERSHEET_REFS}"
-			(at 39.4086 34.29 0)
+			(at 74.9686 49.53 0)
 			(effects
 				(font
@@
 	(hierarchical_label "OUTS"
 		(shape input)
-		(at 64.77 43.18 0)
+		(at 100.33 58.42 0)
 		(effects
 			(font
@@
 	(symbol
 		(lib_id "power:GND")
-		(at 53.34 53.34 0)
+		(at 88.9 68.58 0)
 		(unit 1)
 		(exclude_from_sim no)
@@
 		(dnp no)
 		(fields_autoplaced yes)
-		(property "Reference" "#PWR01"
-			(at 53.34 59.69 0)
+		(property "Reference" "#PWR?"
+			(at 88.9 74.93 0)
 			(effects
 				(font
@@
 		)
 		(property "Value" "GND"
-			(at 53.34 58.42 0)
+			(at 88.9 73.66 0)
 			(effects
 				(font
@@
 		)
 		(property "Footprint" ""
-			(at 53.34 53.34 0)
+			(at 88.9 68.58 0)
 			(effects
 				(font
@@
 		)
 		(property "Datasheet" ""
-			(at 53.34 53.34 0)
+			(at 88.9 68.58 0)
 			(effects
 				(font
@@
 		)
 		(property "Description" "Power symbol creates a global label with name \"GND\" , ground"
-			(at 53.34 53.34 0)
+			(at 88.9 68.58 0)
 			(effects
 				(font
@@
 		)
 		(instances
+			(project "voltage_simulator"
+				(path "/3c45fa24-4483-4d67-9a77-346d2b46feda"
+					(reference "#PWR01")
+					(unit 1)
+				)
+			)
 			(project "Ecu"
-				(path "/c4cd18fd-e378-4fd5-a92c-c83bb44c2a2c/09827d41-bc05-4b52-aa53-b47c66e81042"
-					(reference "#PWR010")
-					(unit 1)
-				)
-				(path "/c4cd18fd-e378-4fd5-a92c-c83bb44c2a2c/1d48189e-f82f-46c2-ab12-d95661aa16cc"
-					(reference "#PWR09")
-					(unit 1)
-				)
-				(path "/c4cd18fd-e378-4fd5-a92c-c83bb44c2a2c/1e064f37-7c9b-4368-9956-5a66bd958fc1"
-					(reference "#PWR011")
-					(unit 1)
-				)
-				(path "/c4cd18fd-e378-4fd5-a92c-c83bb44c2a2c/5875475c-41d9-4569-a0bd-40ef2b754df4"
-					(reference "#PWR01")
-					(unit 1)
-				)
-				(path "/c4cd18fd-e378-4fd5-a92c-c83bb44c2a2c/5e83312d-ee0c-4c56-ad21-a6f5e0f3d810"
-					(reference "#PWR013")
-					(unit 1)
-				)
-				(path "/c4cd18fd-e378-4fd5-a92c-c83bb44c2a2c/9afcdb15-7384-43bf-b426-50def0567352"
-					(reference "#PWR012")
+				(path "/c4cd18fd-e378-4fd5-a92c-c83bb44c2a2c/6f9c8556-2204-4993-a002-1dd36323d11d"
+					(reference "#PWR?")
 					(unit 1)
 				)
@@
 	(symbol
 		(lib_id "Device:R_Potentiometer")
-		(at 53.34 43.18 0)
+		(at 88.9 58.42 0)
 		(unit 1)
 		(exclude_from_sim no)
@@
 		(dnp no)
 		(fields_autoplaced yes)
-		(property "Reference" "RV1"
-			(at 50.8 41.9099 0)
+		(property "Reference" "RV?"
+			(at 86.36 57.1499 0)
 			(effects
 				(font
@@
 		)
 		(property "Value" "R_Potentiometer"
-			(at 50.8 44.4499 0)
+			(at 86.36 59.6899 0)
 			(effects
 				(font
@@
 		)
 		(property "Footprint" "Potentiometer_THT:Potentiometer_Alpha_RD901F-40-00D_Single_Vertical_CircularHoles"
-			(at 53.34 43.18 0)
+			(at 88.9 58.42 0)
 			(effects
 				(font
@@
 		)
 		(property "Datasheet" "~"
-			(at 53.34 43.18 0)
+			(at 88.9 58.42 0)
 			(effects
 				(font
@@
 		)
 		(property "Description" "Potentiometer"
-			(at 53.34 43.18 0)
+			(at 88.9 58.42 0)
 			(effects
 				(font
@@
 		)
 		(instances
+			(project "voltage_simulator"
+				(path "/3c45fa24-4483-4d67-9a77-346d2b46feda"
+					(reference "RV1")
+					(unit 1)
+				)
+			)
 			(project "Ecu"
-				(path "/c4cd18fd-e378-4fd5-a92c-c83bb44c2a2c/09827d41-bc05-4b52-aa53-b47c66e81042"
-					(reference "RV3")
-					(unit 1)
-				)
-				(path "/c4cd18fd-e378-4fd5-a92c-c83bb44c2a2c/1d48189e-f82f-46c2-ab12-d95661aa16cc"
-					(reference "RV2")
-					(unit 1)
-				)
-				(path "/c4cd18fd-e378-4fd5-a92c-c83bb44c2a2c/1e064f37-7c9b-4368-9956-5a66bd958fc1"
-					(reference "RV4")
-					(unit 1)
-				)
-				(path "/c4cd18fd-e378-4fd5-a92c-c83bb44c2a2c/5875475c-41d9-4569-a0bd-40ef2b754df4"
-					(reference "RV1")
-					(unit 1)
-				)
-				(path "/c4cd18fd-e378-4fd5-a92c-c83bb44c2a2c/5e83312d-ee0c-4c56-ad21-a6f5e0f3d810"
-					(reference "RV6")
-					(unit 1)
-				)
-				(path "/c4cd18fd-e378-4fd5-a92c-c83bb44c2a2c/9afcdb15-7384-43bf-b426-50def0567352"
-					(reference "RV5")
-					(unit 1)
-				)
-			)
-		)
-	)
+				(path "/c4cd18fd-e378-4fd5-a92c-c83bb44c2a2c/6f9c8556-2204-4993-a002-1dd36323d11d"
+					(reference "RV?")
+					(unit 1)
+				)
+			)
+		)
+	)
+	(sheet_instances
+		(path "/"
+			(page "1")
+		)
+	)
+	(embedded_fonts no)
 )
